File: pcbs/Logitech_Pedal_Shield_Pro_Micro/Logitech_Pedal_Shield_Pro_Micro.kicad_pcb (KiCad board)
At the start: 2 copper layers, 31.2 x 48.1 mm, 17 parts, among them J1 DE9_Receptacle_MountingHoles, J2 AVR-ISP-6, U1 SparkFun_ProMicro

Commit message: Pedals: Update PCB version to v2.0.0
Matching the shifter, just so that the major repo version matches the PCB version to avoid confusion. No functional changes.
Parts:
- removed kibuzzard-61EDBF18: G***, kibuzzard-61EDBF18
- added G***: LOGO, Sim_Racing_Shields:Version_2.0.0, B.Cu at (152.4, 117.5)
