File: pcbs/Logitech_Shifter_Shield_Pro_Micro/Logitech_Shifter_Shield_Pro_Micro.kicad_pcb (KiCad board)
At the start: 2 copper layers, 31.2 x 48.1 mm, 18 parts, among them J1 DB9_Male_MountingHoles, J2 AVR-ISP-6, U1 SparkFun_ProMicro

Commit message: Update PCBs from schematic (KiCad8)
Bringing in the schematic updates from the new symbols.

No intended functional changes.
Parts:
- J1: value DB9_Male_MountingHoles -> DE9_Plug_MountingHoles
Changed lines of the file:
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@@
 	(net 8 "/Shift_Y")
 	(net 9 "/Shift_Detect")
-	(net 10 "unconnected-(J1-Pad0)")
+	(net 10 "unconnected-(J1-PAD-Pad0)")
 	(net 11 "/MISO")
 	(net 12 "/SCK")
@@
 	(net 15 "/Detect")
 	(net 16 "/CS")
-	(net 17 "unconnected-(U1-Pad1)")
-	(net 18 "unconnected-(U1-Pad2)")
-	(net 19 "unconnected-(U1-Pad5)")
-	(net 20 "unconnected-(U1-Pad6)")
-	(net 21 "unconnected-(U1-Pad7)")
-	(net 22 "unconnected-(U1-Pad8)")
-	(net 23 "unconnected-(U1-Pad9)")
-	(net 24 "unconnected-(U1-Pad10)")
-	(net 25 "unconnected-(U1-Pad11)")
-	(net 26 "unconnected-(U1-Pad12)")
-	(net 27 "unconnected-(U1-Pad20)")
-	(net 28 "unconnected-(U1-Pad24)")
+	(net 17 "unconnected-(J1-PAD-Pad0)_1")
+	(net 18 "unconnected-(U1-RAW-Pad24)")
+	(net 19 "unconnected-(U1-5_PC6-Pad8)")
+	(net 20 "unconnected-(U1-0_PD3_TX1_INT3-Pad1)")
+	(net 21 "unconnected-(U1-1_PD2_RX1_INT2-Pad2)")
+	(net 22 "unconnected-(U1-3_PD0_SCL_INT0-Pad6)")
+	(net 23 "unconnected-(U1-9_PB5_A9-Pad12)")
+	(net 24 "unconnected-(U1-8_PB4_A8-Pad11)")
+	(net 25 "unconnected-(U1-PF4_A3-Pad20)")
+	(net 26 "unconnected-(U1-2_PD1_SDA_INT1-Pad5)")
+	(net 27 "unconnected-(U1-6_PD7_A7-Pad9)")
+	(net 28 "unconnected-(U1-7_PE6_INT6-Pad10)")
 	(net 29 "/AX")
 	(net 30 "/AY")
+	(net 31 "unconnected-(U1-4_PD4_A6-Pad7)")
 	(footprint "kibuzzard-61EDBB73"
 		(layer "F.Cu")
@@
 			)
 		)
-		(property "Value" "DB9_Male_MountingHoles"
+		(property "Value" "DE9_Plug_MountingHoles"
 			(at 5.54 18.44 0)
 			(layer "F.Fab")
@@
 			)
 		)
-		(property "Description" ""
+		(property "Description" "9-pin male plug pin D-SUB connector, Mounting Hole"
 			(at 0 0 0)
 			(layer "F.Fab")
@@
 			)
 		)
+		(property ki_fp_filters "DSUB*Male*")
+		(sheetname "Root")
 		(sheetfile "Logitech_Shifter_Shield_Pro_Micro.kicad_sch")
 		(attr through_hole)
@@
 			(layers "*.Cu" "*.Mask")
 			(remove_unused_layers no)
-			(net 10 "unconnected-(J1-Pad0)")
+			(net 10 "unconnected-(J1-PAD-Pad0)")
 			(pinfunction "PAD")
 			(pintype "passive+no_connect")
@@
 			(layers "*.Cu" "*.Mask")
 			(remove_unused_layers no)
-			(net 10 "unconnected-(J1-Pad0)")
+			(net 17 "unconnected-(J1-PAD-Pad0)_1")
 			(pinfunction "PAD")
 			(pintype "passive+no_connect")
@@
 			)
 		)
+		(property ki_fp_filters "R_*")
+		(sheetname "Root")
 		(sheetfile "Logitech_Shifter_Shield_Pro_Micro.kicad_sch")
 		(attr smd)
@@
 			)
 		)
+		(property ki_fp_filters "R_*")
+		(sheetname "Root")
 		(sheetfile "Logitech_Shifter_Shield_Pro_Micro.kicad_sch")
 		(attr smd)
@@
 			)
 		)
-		(property "Datasheet" ""
+		(property "Datasheet" "https://github.com/sparkfun/Pro_Micro"
 			(at 0 0 0)
 			(layer "F.Fab")
@@
 			)
 		)
+		(sheetname "Root")
 		(sheetfile "Logitech_Shifter_Shield_Pro_Micro.kicad_sch")
 		(attr through_hole)
@@
 			(layers "*.Cu" "*.Mask")
 			(remove_unused_layers no)
-			(net 17 "unconnected-(U1-Pad1)")
+			(net 20 "unconnected-(U1-0_PD3_TX1_INT3-Pad1)")
 			(pinfunction "0_PD3_TX1_INT3")
 			(pintype "bidirectional+no_connect")
@@
 			(layers "*.Cu" "*.Mask")
 			(remove_unused_layers no)
-			(net 18 "unconnected-(U1-Pad2)")
+			(net 21 "unconnected-(U1-1_PD2_RX1_INT2-Pad2)")
 			(pinfunction "1_PD2_RX1_INT2")
 			(pintype "bidirectional+no_connect")
@@
 			(layers "*.Cu" "*.Mask")
 			(remove_unused_layers no)
-			(net 19 "unconnected-(U1-Pad5)")
+			(net 26 "unconnected-(U1-2_PD1_SDA_INT1-Pad5)")
 			(pinfunction "2_PD1_SDA_INT1")
 			(pintype "bidirectional+no_connect")
@@
 			(layers "*.Cu" "*.Mask")
 			(remove_unused_layers no)
-			(net 20 "unconnected-(U1-Pad6)")
+			(net 22 "unconnected-(U1-3_PD0_SCL_INT0-Pad6)")
 			(pinfunction "3_PD0_SCL_INT0")
 			(pintype "bidirectional+no_connect")
@@
 			(layers "*.Cu" "*.Mask")
 			(remove_unused_layers no)
-			(net 21 "unconnected-(U1-Pad7)")
+			(net 31 "unconnected-(U1-4_PD4_A6-Pad7)")
 			(pinfunction "4_PD4_A6")
 			(pintype "bidirectional+no_connect")
@@
 			(layers "*.Cu" "*.Mask")
 			(remove_unused_layers no)
-			(net 22 "unconnected-(U1-Pad8)")
+			(net 19 "unconnected-(U1-5_PC6-Pad8)")
 			(pinfunction "5_PC6")
 			(pintype "bidirectional+no_connect")
@@
 			(layers "*.Cu" "*.Mask")
 			(remove_unused_layers no)
-			(net 23 "unconnected-(U1-Pad9)")
+			(net 27 "unconnected-(U1-6_PD7_A7-Pad9)")
 			(pinfunction "6_PD7_A7")
 			(pintype "bidirectional+no_connect")
@@
 			(layers "*.Cu" "*.Mask")
 			(remove_unused_layers no)
-			(net 24 "unconnected-(U1-Pad10)")
+			(net 28 "unconnected-(U1-7_PE6_INT6-Pad10)")
 			(pinfunction "7_PE6_INT6")
 			(pintype "bidirectional+no_connect")
@@
 			(layers "*.Cu" "*.Mask")
 			(remove_unused_layers no)
-			(net 25 "unconnected-(U1-Pad11)")
+			(net 24 "unconnected-(U1-8_PB4_A8-Pad11)")
 			(pinfunction "8_PB4_A8")
 			(pintype "bidirectional+no_connect")
@@
 			(layers "*.Cu" "*.Mask")
 			(remove_unused_layers no)
-			(net 26 "unconnected-(U1-Pad12)")
+			(net 23 "unconnected-(U1-9_PB5_A9-Pad12)")
 			(pinfunction "9_PB5_A9")
 			(pintype "bidirectional+no_connect")
@@
 			(layers "*.Cu" "*.Mask")
 			(remove_unused_layers no)
-			(net 27 "unconnected-(U1-Pad20)")
+			(net 25 "unconnected-(U1-PF4_A3-Pad20)")
 			(pinfunction "PF4_A3")
 			(pintype "bidirectional+no_connect")
@@
 			(layers "*.Cu" "*.Mask")
 			(remove_unused_layers no)
-			(net 28 "unconnected-(U1-Pad24)")
+			(net 18 "unconnected-(U1-RAW-Pad24)")
 			(pinfunction "RAW")
 			(pintype "power_in+no_connect")
@@
 			)
 		)
+		(property ki_fp_filters "Jumper* TestPoint*2Pads* TestPoint*Bridge*")
+		(sheetname "Root")
 		(sheetfile "Logitech_Shifter_Shield_Pro_Micro.kicad_sch")
 		(attr exclude_from_pos_files exclude_from_bom)
@@
 			)
 		)
+		(property ki_fp_filters "Jumper* TestPoint*2Pads* TestPoint*Bridge*")
+		(sheetname "Root")
 		(sheetfile "Logitech_Shifter_Shield_Pro_Micro.kicad_sch")
 		(attr exclude_from_pos_files exclude_from_bom)
@@
 			)
 		)
+		(property ki_fp_filters "Jumper* TestPoint*2Pads* TestPoint*Bridge*")
+		(sheetname "Root")
 		(sheetfile "Logitech_Shifter_Shield_Pro_Micro.kicad_sch")
 		(attr exclude_from_pos_files exclude_from_bom)
@@
 			)
 		)
+		(property ki_fp_filters "Jumper* TestPoint*2Pads* TestPoint*Bridge*")
+		(sheetname "Root")
 		(sheetfile "Logitech_Shifter_Shield_Pro_Micro.kicad_sch")
 		(attr exclude_from_pos_files exclude_from_bom)
@@
 			)
 		)
+		(property ki_fp_filters "Jumper* TestPoint*2Pads* TestPoint*Bridge*")
+		(sheetname "Root")
 		(sheetfile "Logitech_Shifter_Shield_Pro_Micro.kicad_sch")
 		(attr exclude_from_pos_files exclude_from_bom)
@@
 			)
 		)
+		(property ki_fp_filters "Jumper* TestPoint*2Pads* TestPoint*Bridge*")
+		(sheetname "Root")
 		(sheetfile "Logitech_Shifter_Shield_Pro_Micro.kicad_sch")
 		(attr exclude_from_pos_files exclude_from_bom)
@@
 			)
 		)
+		(property ki_fp_filters "Jumper* TestPoint*2Pads* TestPoint*Bridge*")
+		(sheetname "Root")
 		(sheetfile "Logitech_Shifter_Shield_Pro_Micro.kicad_sch")
 		(attr exclude_from_pos_files exclude_from_bom)
@@
 			)
 		)
-		(property "Description" ""
+		(property "Description" "Atmel 6-pin ISP connector"
 			(at 0 0 -90)
 			(layer "F.Fab")
@@
 			)
 		)
+		(property ki_fp_filters "IDC?Header*2x03* Pin?Header*2x03*")
+		(sheetname "Root")
 		(sheetfile "Logitech_Shifter_Shield_Pro_Micro.kicad_sch")
 		(attr exclude_from_pos_files)
