File: pcbs/Logitech_Shifter_Shield_Pro_Micro/Logitech_Shifter_Shield_Pro_Micro.kicad_pcb (KiCad board)
At the start: 2 copper layers, 31.2 x 48.1 mm, 18 parts, among them J1 DB9_Male_MountingHoles, J2 AVR-ISP-6, U1 SparkFun_ProMicro

Commit message: KiCad 8 Format Updates (#4)
* Add KiCad files to gitignore
* Update PCBs to KiCad8 format (8.0.8)
* Relink DE-9 connector symbols
* Update modified schematic symbols
* Pedals: Fix 'wire off grid' schematic error
* Set min_copper_edge_clearance
* Update PCBs from schematic

This updates the format of the PCB files to be compatible with KiCad 8 There are no intended functional changes.
Parts:
- J1: value DB9_Male_MountingHoles -> DE9_Plug_MountingHoles
