File: pcbs/Logitech_Shifter_Shield_Pro_Micro/Logitech_Shifter_Shield_Pro_Micro.kicad_sch (KiCad schematic)
At the start: 12 parts, among them J1 DB9_Male_MountingHoles, J2 AVR-ISP-6, U1 SparkFun_ProMicro

Commit message: KiCad 8 Format Updates (#4)
* Add KiCad files to gitignore
* Update PCBs to KiCad8 format (8.0.8)
* Relink DE-9 connector symbols
* Update modified schematic symbols
* Pedals: Fix 'wire off grid' schematic error
* Set min_copper_edge_clearance
* Update PCBs from schematic

This updates the format of the PCB files to be compatible with KiCad 8 There are no intended functional changes.
Parts:
- J1: value DB9_Male_MountingHoles -> DE9_Plug_MountingHoles; symbol Connector:DB9_Male_MountingHoles -> Connector:DE9_Plug_MountingHoles
- JP1, JP2, JP3, JP5: footprint (none) -> Sim_Racing_Shields:SolderJumper-2_P1.3mm_Bridged_RoundedPad1.0x1.5mm_Unmasked
- U1: footprint (none) -> Sim_Racing_Shields:Sparkfun_ProMicro
Other:
- note added: "DE9 Male Port"
- note removed: "DB9 Male Port"

Commit message: Bill of Materials (BOM) (#5)
Adds Bill of Materials (BOM) information to the KiCad schematic, which can be exported to CSV using the "Generate Bill of Materials" option in the toolbar of the schematic editor.

These parts are, to the best of my knowledge, the parts I used when assembling these boards two and a half years ago. You do not need to use these exact parts, substitutes may be available that are currently stocked and/or less expensive. The 1% resistors, in particular, do not need to be tight tolerance - that's just what I had on hand.
Parts:
- J1: DigiKey Part Number (none) -> AE10968-ND; Manufacturer (none) -> Assmann WSW Components; Part Number (none) -> A-DS 09 A/KG-T2S
- J2: now left out of the parts list
- R1, R2: DigiKey Part Number (none) -> YAG1319CT-ND; Manufacturer (none) -> YAGEO; Part Number (none) -> RC0805FR-0710KP
- U1: DigiKey Part Number (none) -> 1568-DEV-15795-ND; Manufacturer (none) -> SparkFun Electronics; Part Number (none) -> DEV-15795
